File: MAX14748_Demo.kicad_sch (KiCad schematic)
At the start: 36 parts, among them IC1 MAX14748BEWW+T, IC3 NC7WZ07P6X, IC4 NC7WZ07P6X, J1 USB_C_Receptacle_USB2.0_16P, J10 Conn_01x02, J2 Conn_01x02, J3 Conn_01x02, J4 Conn_01x02, J5 Conn_01x02, J6 Conn_02x06_Counter_Clockwise, J7 Conn_01x03, J8 Conn_01x03, J9 Conn_01x02, SW1 SW_Push

Commit message: Update Modify
Change-Id: I3a529a3a4b0c42d914bed02b21a5350ab12660de
Parts:
- added C10, C15, C6, C8: 22uf, symbol Device:C
- added C11, C12, C5: 1uf, symbol Device:C
- added C13, C14: 10uf, symbol Device:C
- added C16, C18, C7, C9: 0.1uf, symbol Device:C
- added C17: 3900pf, symbol Device:C
- added D6: GREEN, symbol Device:LED
- added J11, J12, J13, J14, J16: Conn_01x02, symbol Connector_Generic:Conn_01x02
- added J15: Conn_02x02_Odd_Even, symbol Connector_Generic:Conn_02x02_Odd_Even
- added L1: 2.2uh, symbol Device:L
- added Q2: RRL035P03TR, RRL035P03TR, symbol MAX14748_Demo:RRL035P03TR
- added R15: 499, symbol Device:R
- added R16: 10k, symbol Device:R
- added R17: 100k, symbol Device:R
- added RV2: 100k, symbol Device:R_Potentiometer
- added TP2, TP3, TP4, TP5, TP6, TP7, TP8, TP9: TestPoint, symbol Connector:TestPoint
Connections:
- net CDIR: now also IC1.E5 (CDIR)
- net FLTIN: now also IC1.A2 (~{FLTIN})
- net GND: now also IC1.A1 (AGND), IC1.B3 (DGND), IC1.C4 (GND_1), IC1.D4 (GND_2), IC1.D5 (GND_3), IC1.D6 (PGND_1), IC1.D7 (PGND_2), IC1.D8 (PGND_3), IC1.D9 (PGND_4), J1.A1 (GND), J1.A12 (GND), J1.B1 (GND), J1.B12 (GND), J1.S1 (SHIELD), C10.2, C11.2, C12.2, C13.2, C14.2, C15.2, C16.2, C17.1, C5.2, C6.2, C7.2, C8.2, C9.2, J11.1 (Pin_1), R17.2, RV2.1
- net INT: now also IC1.D3 (~{INT})
- net SCL: now also IC1.C2 (SCL)
- net SDA: now also IC1.D2 (SDA)
- net SET: now also IC1.A6 (SET)
- net SYSOK: now also IC1.A3 (SYSOK)
- net VIO: now also D6.2 (A), J16.2 (Pin_2)
- net TPU: now reaches IC1.A4 (TPU)
- net TPU: now also R16.1
- net at IC1.A5 (COMP): now also C17.2
- net BAT: now reaches IC1.A7 (BAT_1)
- net BAT: now also IC1.A8 (BAT_2), IC1.A9 (BAT_3), C15.1, C16.1, J11.2 (Pin_2), TP9.1
- net CC2: now reaches IC1.B1 (CC2)
- net CC2: now also J1.B5 (CC2)
- net FSUS: now reaches IC1.B2 (FSUS)
- net FSUS: now also J16.1 (Pin_1), R17.1
- net VTPU: now reaches IC1.B4 (VTPU)
- net VTPU: now also J14.2 (Pin_2)
- net BREG: now reaches IC1.B5 (BREG)
- net BREG: now also C13.1, TP7.1
- net SYS: now reaches IC1.B6 (SYS_1)
- net SYS: now also IC1.B7 (SYS_2), IC1.B8 (SYS_3), IC1.B9 (SYS_4), C10.1, C8.1, C9.1, TP4.1
- net VCCINT: now reaches IC1.C3 (VCCINT)
- net VCCINT: now also C14.1, J14.1 (Pin_1), TP8.1
- net at IC1.C5 (BST): now also C18.2
- net at IC1.C6 (LX_1): now also IC1.C7 (LX_2), IC1.C8 (LX_3), IC1.C9 (LX_4), C18.1, L1.2
- net CC1: now reaches IC1.D1 (CC1)
- net CC1: now also J1.A5 (CC1)
- net CND: now reaches IC1.E1 (CDN)
- net at IC1.E2 (LED): now also R15.1
- net THM: now reaches IC1.E3 (THM)
- net THM: now also J12.1 (Pin_1), J13.2 (Pin_2)
- net FOUT: now reaches IC1.E4 (SFOUT)
- net BYP: now reaches IC1.E6 (BYP_1)
- net BYP: now also IC1.E7 (BYP_2), IC1.E8 (BYP_3), IC1.E9 (BYP_4), C6.1, C7.1, L1.1, TP3.1
- net CDP: now reaches IC1.F1 (CDP)
- net CDP: now also J1.A6 (D+), J1.B6 (D+)
- net BVCEN: now reaches IC1.F4 (BVCEN)
- net NVP: now reaches IC1.F5 (NVP)
- net NVP: now also Q2.3 (GATE)
- net CHGIN: now reaches IC1.F6 (CHGIN_1)
- net CHGIN: now also IC1.F7 (CHGIN_2), IC1.F8 (CHGIN_3), IC1.F9 (CHGIN_4), C12.1, J15.2 (Pin_2), J15.4 (Pin_4), TP6.1
- net VUSB_C: now reaches J1.A4 (VBUS), J1.A9 (VBUS), J1.B4 (VBUS), J1.B9 (VBUS)
- net VUSB_C: now also C5.1, Q2.1 (DRAIN_1), Q2.2 (DRAIN_2), Q2.5 (DRAIN_3), Q2.6 (DRAIN_4), TP2.1
- net CDN: now reaches J1.A7 (D-)
- net CDN: now also J1.B7 (D-)
- net SBU1: now reaches J1.A8 (SBU1)
- net SBU2: now reaches J1.B8 (SBU2)
- new net: J12.2 (Pin_2), R16.2
- new net: J15.1 (Pin_1), J15.3 (Pin_3), Q2.4 (SOURCE)
- new net: D6.1 (K), R15.2
- new net: J13.1 (Pin_1), RV2.2, RV2.3
- new net SFOUT: C11.1, TP5.1
Other:
- moved on the sheet: IC1

Commit message: Modify Update
Change-Id: If6ab4a9ec106b7a63e2a49d27166ab09263834bd
Parts:
- added IC2: NX5P2924DUKZ, MAX14748_Demo:BGA6C50P2X3_89X139X50, symbol MAX14748_Demo:NX5P2924DUKZ
- added J17: USB_B_Mini, symbol Connector:USB_B_Mini
- added R18: 1K, symbol Device:R
- added TP18: TP18, symbol Connector:TestPoint
- added TP19: TP19, symbol Connector:TestPoint
- C13, C14: value 10uf -> 1uf
- C4: value 0.1uf -> 1uf
- IC1: footprint BGA54C40P9X6_397X277X69 -> MAX14748_Demo:BGA54C40P9X6_397X277X69
- IC3, IC4: footprint SOT65P210X110-6N -> MAX14748_Demo:SOT65P210X110-6N
- Q2: footprint RRL035P03TR -> MAX14748_Demo:RRL035P03TR
- TP0: renamed from TP1; value TestPoint -> TP0
- TP1: renamed from TP9; value TestPoint -> TP1
- TP2: value TestPoint -> TP2
- TP3: value TestPoint -> TP3
- TP4: value TestPoint -> TP4
- TP5: value TestPoint -> TP5
- TP6: value TestPoint -> TP6
- TP7: value TestPoint -> TP7
- TP8: value TestPoint -> TP8
Connections:
- net CND is gone; now on net CDN: IC1.E1 (CDN)
- net FOUT is gone; now on net SFOUT: IC1.E4 (SFOUT)
- net BVCEN: now also R18.2
- net GND: now also IC2.C1 (GND), J17.5 (GND), J17.6 (Shield)
- net VUSB_C: now also J17.1 (VBUS)
- net VCONN: now reaches IC1.C1 (VCONN)
- net VCONN: now also IC2.A1 (VOUT_1), IC2.B1 (VOUT_2), TP18.1
- net TDP: now reaches IC1.F2 (TDP)
- net TDP: now also J17.3 (D+)
- net TDN: now reaches IC1.F3 (TDN)
- net TDN: now also J17.2 (D-)
- net SBU1: no longer names the net of J1.A8 (SBU1)
- net SBU2: no longer names the net of J1.B8 (SBU2)
- new net: IC2.A2 (VIN_1), IC2.B2 (VIN_2), TP19.1
- new net: IC2.C2 (EN), R18.1
- no-connect marks 0 -> 9
Other:
- moved on the sheet: C17, C18, D6, IC1, L1, R15
